File: PCBs/checkin-tiny/wifi.brd (EAGLE design)
At the start: 62.5 x 36.7 mm, 23 parts, among them IC1 Primary, IC2 Display, Q1 12 MHz, Q2 12 MHz

Commit message: Fix resistor labels on Wi-Fi board
Parts:
- R1, R2: value (none) -> 10K
Changed lines of the file:
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@@
 <attribute name="VALUE" x="8.128" y="2.159" size="0.762" layer="27" ratio="10" rot="R180"/>
 </element>
-<element name="R1" library="rcl" library_urn="urn:adsk.eagle:library:334" package="R1206" package3d_urn="urn:adsk.eagle:package:23540/2" value="" x="30.48" y="-5.08" smashed="yes" rot="R90">
+<element name="R1" library="rcl" library_urn="urn:adsk.eagle:library:334" package="R1206" package3d_urn="urn:adsk.eagle:package:23540/2" value="10K" x="30.48" y="-5.08" smashed="yes" rot="R90">
 <attribute name="NAME" x="29.3116" y="-7.0866" size="0.762" layer="25" ratio="10" rot="R90"/>
 <attribute name="POPULARITY" value="19" x="30.48" y="-5.08" size="1.778" layer="27" rot="R90" display="off"/>
@@
 <attribute name="VALUE" x="32.7914" y="-7.2136" size="0.9906" layer="27" ratio="10" rot="R90"/>
 </element>
-<element name="R2" library="rcl" library_urn="urn:adsk.eagle:library:334" package="R1206" package3d_urn="urn:adsk.eagle:package:23540/2" value="" x="19.05" y="-5.08" smashed="yes" rot="R90">
+<element name="R2" library="rcl" library_urn="urn:adsk.eagle:library:334" package="R1206" package3d_urn="urn:adsk.eagle:package:23540/2" value="10K" x="19.05" y="-5.08" smashed="yes" rot="R90">
 <attribute name="NAME" x="19.6596" y="-7.7724" size="0.762" layer="25" ratio="10" rot="R180"/>
 <attribute name="POPULARITY" value="19" x="19.05" y="-5.08" size="1.778" layer="27" rot="R90" display="off"/>
